File: hardware/SC_Detection.kicad_sch (KiCad schematic)
At the start: 86 parts, among them U15 LT1678CS8#PBF, U16 LT1678CS8#PBF, U17 LM211DRG4, U18 LM211DRG4, U19 LM211DRG4, U20 LM211DRG4

Commit message: The final review has been completed, and the manufacturing files have been generated.
Parts:
- C60, C61, C62, C63, C80, C81, C82, C83: MPN C0603C150K5RACTU -> (none)
- C64, C65, C66, C67, C68, C69, C70, C71, C72, C73, C74, C75, C76, C77, C78, C79, C84, C85, C86, C87, C88, C89, C90, C91: MPN C0603C104K5RACTU -> (none)
- D1, D2, D3, D4: MPN BAT43W-7-F -> (none)
- R42, R43, R44, R45, R78, R79, R80, R81: MPN RT0603BRD074K02L -> (none)
- R46, R47, R48, R49, R70, R71, R72, R73: MPN RT0603BRD0740K2L -> (none)
- R50, R51, R52, R53: MPN RC0603FR-07100KL -> (none)
- R54, R55, R56, R57, R58, R59, R60, R61: MPN RT0603BRD074K75L -> (none)
- R62, R64, R66, R68: MPN RT0603BRD0747K5L -> (none)
- R63, R65, R67, R69, R82, R83, R84, R85: MPN RT0603BRD0710KL -> (none)
- R74, R75, R76, R77: MPN AC0603FR-1310RL -> (none)
- U15, U16: MPN LT1678CS8#PBF -> (none)
- U17, U18, U19, U20: MPN LM211DRG4 -> (none)
