File: hardware/Communication.kicad_sch (KiCad schematic)
At the start: 28 parts, among them J1 Conn_01x04_Pin, J2 Conn_01x03_Male, J3 USB_C_Receptacle_USB2.0, U21 TXB0102DCUT, U22 ADUM4160

Commit message: The final review has been completed, and the manufacturing files have been generated.
Parts:
- C92, C93, C94, C97: MPN C0603C104K5RACTU -> (none)
- C95, C96: MPN C1608X7R1H105K080AB -> (none)
- J1: MPN n/a -> (none); Manufacturer_Name n/a -> SAMTEC; Manufacturer_Part_Number n/a -> TSW-104-07-G-S
- J2: value Conn_01x03_Male -> 5-146281-3; MPN n/a -> (none); Manufacturer_Name n/a -> TE Connectivity; Manufacturer_Part_Number n/a -> 5-146281-3
- J3: MPN DX07S016JA1R1500 -> (none)
- LED8: MFN SunLED -> (none); MPN XZCDGK53W-1VF -> (none); Manufacturer_Name SunLED -> Vishay; Manufacturer_Part_Number XZCDGK53W-1VF -> VLMTG1300-GS08
- R86, R88, R89: MPN RC0603JR-070RL -> (none)
- R87: MPN RC0603FR-07100KL -> (none)
- R90: MPN RC0603FR-07330RL -> (none)
- R91, R92: MPN RC0603FR-075K1L -> (none)
- R93, R94, R95, R96: MPN AC0603FR-0724RL -> (none)
- TVS1, TVS3, TVS5: MPN ESD441DPLR -> (none)
- TVS2: MPN CDDFN10-3324P -> (none)
- TVS4: MPN TPD2EUSB30DRTR -> (none)
- U21: MPN TXB0102DCUT -> (none)
- U22: MPN ADUM4160BRWZ-RL -> (none)
