File: hardware/Communication.kicad_sch (KiCad schematic)
At the start: 28 parts, among them J1 Conn_01x04_Pin, J2 5-146281-3, J3 USB_C_Receptacle_USB2.0, U21 TXB0102DCUT, U22 ADUM4160

Commit message: Some improvements have been made to the layout.
Parts:
- renumbered J2 to J17, J1 to J18
Changed lines of the file:
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@@
 		(on_board yes)
 		(dnp no)
-		(property "Reference" "J1"
+		(property "Reference" "J18"
 			(at 35.56 22.098 0)
 			(effects
@@
 			(project "harp.device.quad.dac"
 				(path "/6b47c519-21c4-43bd-9777-b273999e4447/08506a40-9943-41e4-b528-13f6a4c7e855"
-					(reference "J1")
+					(reference "J18")
 					(unit 1)
 				)
@@
 		(on_board yes)
 		(dnp no)
-		(property "Reference" "J2"
+		(property "Reference" "J17"
 			(at 37.084 62.484 0)
 			(effects
@@
 			(project "harp.device.quad.dac"
 				(path "/6b47c519-21c4-43bd-9777-b273999e4447/08506a40-9943-41e4-b528-13f6a4c7e855"
-					(reference "J2")
-					(unit 1)
-				)
+					(reference "J17")
+					(unit 1)
+				)
