File: hardware/DACs.kicad_sch (KiCad schematic)
At the start: 70 parts, among them U10 LT1678CS8#PBF, U11 LT1678CS8#PBF, U12 LT1678CS8#PBF, U13 LT1678CS8#PBF, U14 LT1461CIS8-2.5#PBF, U6 LTC2642ACDD-16#PBF, U7 LTC2642ACDD-16#PBF, U8 LTC2642ACDD-16#PBF, U9 LTC2642ACDD-16#PBF

Commit message: The final review has been completed, and the manufacturing files have been generated.
Parts:
- C30, C32, C33, C34, C35, C37, C39, C40, C41, C42, C44, C45, C46, C47, C49: MPN C0603C104K5RACTU -> (none)
- C31, C38, C43, C48: MPN C1608X7R1H105K080AB -> (none)
- C36, C58, C59: MPN GRM188R61E106KA73D -> (none)
- C50, C51, C52, C53, C54, C55, C56, C57: MPN C0603C150K5RACTU -> (none)
- LED4, LED5, LED6, LED7: MFN SunLED -> (none); MPN XZCDGK53W-1VF -> (none); Manufacturer_Name SunLED -> Vishay; Manufacturer_Part_Number XZCDGK53W-1VF -> VLMTG1300-GS08
- R19, R20, R21, R22: MPN RC0603FR-07330RL -> (none)
- R23, R24: MPN RC0603JR-070RL -> (none)
- R25: MPN AC0603FR-13100RL -> (none)
- R26, R27, R28, R29, R30, R31, R32, R33: MPN RT0603BRD0740K2L -> (none)
- R34, R35, R36, R37, R38, R39, R40, R41: MPN RT0603BRD0710KL -> (none)
- RSh1, RSh2, RSh3, RSh4: MPN RCG120610R0FKEA -> (none); Manufacturer_Part_Number CRCW120610R0FKEBC -> RCG120610R0FKEA
- U10, U11, U12, U13: MPN LT1678CS8#PBF -> (none)
- U14: MPN LT1461CIS8-2.5#PBF -> (none)
- U6, U7, U8, U9: MPN LTC2642ACDD-16#PBF -> (none)
