File: hardware/Output.kicad_sch (KiCad schematic)
At the start: 26 parts, among them J11 Conn_Coaxial, J12 Conn_Coaxial, J13 Conn_Coaxial, J14 Conn_Coaxial, J15 Conn_Coaxial, J16 Conn_Coaxial, J17 Conn_Coaxial, J18 Conn_Coaxial, U31 74LVCH2T45DC, U32 74LVCH2T45DC

Commit message: Continue BOM + enhance BOM + enhance schematic
Parts:
- TVS12, TVS13, TVS14, TVS15: Link (none) -> https://www.digikey.com/en/products/detail/texas-instrument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
- TVS16, TVS17, TVS18, TVS19: Link (none) -> https://www.digikey.com/en/products/detail/nexperia-usa-inc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; MPN ESDSB12VLB-TP -> PESD12VL1BSLAZ; Manufacturer MCC -> Nexperia
- U31, U32: MPN (none) -> 74LVCH2T45DC,125; Manufacturer Nexperia USA Inc. -> Nexperia; Manufacturer_Name Nexperia USA Inc. -> Nexperia; Manufacturer_Part_Number (none) -> 74LVCH2T45DC,125
Changed lines of the file:
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@@
 			)
 		)
+		(property "Link" "https://www.digikey.com/en/products/detail/texas-instruments/ESD441DPLR/21298753"
+			(at 110.49 95.25 0)
+			(effects
+				(font
+					(size 1.27 1.27)
+				)
+				(hide yes)
+			)
+		)
 		(pin "2"
 		)
@@
 			)
 		)
+		(property "Link" "https://www.digikey.com/en/products/detail/texas-instruments/ESD441DPLR/21298753"
+			(at 110.49 31.75 0)
+			(effects
+				(font
+					(size 1.27 1.27)
+				)
+				(hide yes)
+			)
+		)
 		(pin "2"
 		)
@@
 			)
 		)
-		(property "Manufacturer" "Nexperia USA Inc."
+		(property "Manufacturer" "Nexperia"
 			(at 74.93 118.11 0)
 			(effects
@@
 			)
 		)
-		(property "Manufacturer_Name" "Nexperia USA Inc."
+		(property "Manufacturer_Name" "Nexperia"
+			(at 74.93 118.11 0)
+			(effects
+				(font
+					(size 1.27 1.27)
+				)
+				(hide yes)
+			)
+		)
+		(property "MPN" "74LVCH2T45DC,125"
+			(at 74.93 118.11 0)
+			(effects
+				(font
+					(size 1.27 1.27)
+				)
+				(hide yes)
+			)
+		)
+		(property "Manufacturer_Part_Number" "74LVCH2T45DC,125"
 			(at 74.93 118.11 0)
 			(effects
@@
 			)
 		)
-		(property "Manufacturer" "Nexperia USA Inc."
+		(property "Manufacturer" "Nexperia"
 			(at 74.93 54.61 0)
 			(effects
@@
 			)
 		)
-		(property "Manufacturer_Name" "Nexperia USA Inc."
+		(property "Manufacturer_Name" "Nexperia"
+			(at 74.93 54.61 0)
+			(effects
+				(font
+					(size 1.27 1.27)
+				)
+				(hide yes)
+			)
+		)
+		(property "MPN" "74LVCH2T45DC,125"
+			(at 74.93 54.61 0)
+			(effects
+				(font
+					(size 1.27 1.27)
+				)
+				(hide yes)
+			)
+		)
+		(property "Manufacturer_Part_Number" "74LVCH2T45DC,125"
 			(at 74.93 54.61 0)
 			(effects
@@
 			)
 		)
+		(property "Link" "https://www.digikey.com/en/products/detail/texas-instruments/ESD441DPLR/21298753"
+			(at 110.49 127 0)
+			(effects
+				(font
+					(size 1.27 1.27)
+				)
+				(hide yes)
+			)
+		)
 		(pin "2"
 		)
@@
 			)
 		)
-		(property "Manufacturer" "MCC"
+		(property "Manufacturer" "Nexperia"
+			(at 184.15 95.25 0)
+			(effects
+				(font
+					(size 1.27 1.27)
+				)
+				(hide yes)
+			)
+		)
+		(property "MPN" "PESD12VL1BSLAZ"
 			(at 184.15 95.25 0)
 			(effects
@@
 			)
 		)
-		(property "MPN" "ESDSB12VLB-TP"
+		(property "Link" "https://www.digikey.com/en/products/detail/nexperia-usa-inc/PESD12VL1BSLAZ/16021611"
 			(at 184.15 95.25 0)
 			(effects
@@
 			)
 		)
-		(property "Manufacturer" "MCC"
+		(property "Manufacturer" "Nexperia"
+			(at 184.15 31.75 0)
+			(effects
+				(font
+					(size 1.27 1.27)
+				)
+				(hide yes)
+			)
+		)
+		(property "MPN" "PESD12VL1BSLAZ"
 			(at 184.15 31.75 0)
 			(effects
@@
 			)
 		)
-		(property "MPN" "ESDSB12VLB-TP"
+		(property "Link" "https://www.digikey.com/en/products/detail/nexperia-usa-inc/PESD12VL1BSLAZ/16021611"
 			(at 184.15 31.75 0)
 			(effects
@@
 			)
 		)
-		(property "Manufacturer" "MCC"
+		(property "Manufacturer" "Nexperia"
 			(at 184.15 127 0)
 			(effects
@@
 			)
 		)
-		(property "MPN" "ESDSB12VLB-TP"
+		(property "MPN" "PESD12VL1BSLAZ"
+			(at 184.15 127 0)
+			(effects
+				(font
+					(size 1.27 1.27)
+				)
+				(hide yes)
+			)
+		)
+		(property "Link" "https://www.digikey.com/en/products/detail/nexperia-usa-inc/PESD12VL1BSLAZ/16021611"
 			(at 184.15 127 0)
 			(effects
@@
 			)
 		)
-		(property "Manufacturer" "MCC"
+		(property "Manufacturer" "Nexperia"
+			(at 184.15 63.5 0)
+			(effects
+				(font
+					(size 1.27 1.27)
+				)
+				(hide yes)
+			)
+		)
+		(property "MPN" "PESD12VL1BSLAZ"
 			(at 184.15 63.5 0)
 			(effects
@@
 			)
 		)
-		(property "MPN" "ESDSB12VLB-TP"
+		(property "Link" "https://www.digikey.com/en/products/detail/nexperia-usa-inc/PESD12VL1BSLAZ/16021611"
 			(at 184.15 63.5 0)
 			(effects
@@
 			(at 110.49 66.04 0)
 			(effects
+				(font
+					(size 1.27 1.27)
+				)
+				(hide yes)
+			)
+		)
+		(property "Link" "https://www.digikey.com/en/products/detail/texas-instruments/ESD441DPLR/21298753"
+			(at 110.49 66.04 0)
+			(effects

Commit message: The final review has been completed, and the manufacturing files have been generated.
Parts:
- C148, C149, C150, C151: MPN C0603C104K5RACTU -> (none)
- J11, J12, J13, J14, J15, J16, J17, J18: MPN CONSMA002-SMD-G-T -> (none)
- R128, R129, R130, R131: MPN AC0603FR-1310RL -> (none)
- TVS12, TVS13, TVS14, TVS15: MPN ESD441DPLR -> (none)
- TVS16, TVS17, TVS18, TVS19: MPN PESD12VL1BSLAZ -> (none)
- U31, U32: MPN 74LVCH2T45DC,125 -> (none)
