File: hardware/Input.kicad_sch (KiCad schematic)
At the start: 40 parts, among them J10 USB_C_Receptacle_USB2.0, J4 AudioJack3, J5 Conn_Coaxial, J6 Conn_Coaxial, J7 Conn_Coaxial, J8 Conn_Coaxial, J9 Barrel_Jack_Switch, U23 74LVCH2T45DC, U24 74LVCH2T45DC, U25 74LVCH2T45DC

Commit message: Some improvements have been made to the layout.
Parts:
- renumbered J10 to J1, J9 to J2, J6 to J5, J5 to J6, J8 to J7, J7 to J8
Connections:
- net at R98.2, TVS6.1: now also U23.3 (2A); no longer U23.2 (1A)
- net at R99.2, TVS7.1: now also U23.2 (1A); no longer U23.3 (2A)
- net at R100.2, TVS8.1: now also U24.3 (2A); no longer U24.2 (1A)
- net at J5.1 (In): now also R100.1; no longer R99.1
- net at R101.1: now also J6.1 (In); no longer J7.1 (In)
- net at R101.2, TVS9.1: now also U24.2 (1A); no longer U24.3 (2A)
- net at R98.1: now also J7.1 (In); no longer J6.1 (In)
- net at J8.1 (In): now also R99.1; no longer R100.1
Other:
- moved on the sheet: J5, J6, J7, J8, R100, R101, R98, R99, TVS6, TVS7, TVS8, TVS9
